File: LED Project/LED Project.kicad_pcb (KiCad board)
At the start: 2 copper layers, 23.5 x 23.5 mm, 3 parts, among them J1 Conn_01x02_Pin

Commit message: ON-OFF-LAMP First Trial
Parts:
- added SW1: SW_MEC_5E, Button_Switch_SMD:SW_SPST_SKQG_WithStem, F.Cu at (51.2, 31.6)
Routing:
- net +3.3V: track 21.7 -> 39.7 mm
- net GND: track 2.86 -> 16.7 mm
Other:
- board size 23.5 x 23.5 mm -> 23.5 x 31.2 mm
